Commit message: Update base_link.urdf

File: base_link.urdf (robot description, URDF)
Before this commit: robot your_robot_name, 1 links, 0 joints
Links:
- link base_link: mass ${base_mass} -> 25; geometry collision box size=0.4 0.4 0.1; visual box size=0.4 0.4 0.1

Commit message: Update base_link.urdf

File: base_link.urdf (robot description, URDF)
Before this commit: robot your_robot_name, 1 links, 0 joints
Links:
- link base_link: mass 25 -> 5
